Commit message: push code for data collection pipeline

File: src/heater_moveit_config/config/gazebo_motoman_gp12.urdf (robot description, URDF)
Before this commit: robot motoman_gp12, 10 links, 9 joints
Links:
- added link heat_gun_tip
Joints:
- added joint heat_gun-heat_gun_tip: type fixed, parent heater_gun, child heat_gun_tip, origin xyz=0 0 -0.300 rpy=0 0 0
